File: Power.kicad_sch (KiCad schematic)
At the start: 0 parts

Commit message: Added user buttons and boot config
Parts:
- added U6: STM32F407VGTx, Package_QFP:LQFP-100_14x14mm_P0.5mm, symbol MCU_ST_STM32F4:STM32F407VGTx
Connections:
- new net: U6.10 (VSS), U6.27 (VSS), U6.74 (VSS), U6.99 (VSS)

Commit message: update
Parts:
- removed U6: STM32F407VGTx, Package_QFP:LQFP-100_14x14mm_P0.5mm, symbol MCU_ST_STM32F4:STM32F407VGTx
