File: Block Diagram.kicad_sch (KiCad schematic)
At the start: 0 parts

Commit message: Initial Review Changes
Other:
- company: (none) -> _electronic_projects
- title: (none) -> DeskNode-F4
Changed lines of the file:
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@@
 	(generator_version "9.0")
 	(paper "A4")
+	(title_block
+		(title "DeskNode-F4")
+		(rev "A")
+		(company "_electronic_projects")
+		(comment 1 "Wajahatulla Sharif")
+		(comment 2 "Designed by ")
+	)
 	(rectangle
 		(start 211.328 90.17)

Commit message: Review files
Other:
- company: _electronic_projects -> (none)
Changed lines of the file:
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@@
 		(title "DeskNode-F4")
 		(rev "A")
-		(company "_electronic_projects")
-		(comment 1 "Wajahatulla Sharif")
-		(comment 2 "Designed by ")
 	)
 	(rectangle
