File: Debugger.kicad_sch (KiCad schematic)
At the start: 33 parts, among them J4 F103 SWD, J5 USB_B_Micro, SW5 SW_Push, U3 STM32F103C8T6, U4 USBLC6-2, Y1 8MHz

Commit message: Alternate MPNs added
Parts:
- F1: MPN NANOSMDC075 -> NANOSMDC075F-2; Manufacturer_Part_Number (none) -> NANOSMDC075
- J5: MPN USB3076-30 -> USB3076-30-A; Manufacturer_Part_Number (none) -> USB3076-30
- TP5: value 5V -> TestPoint
- Y1: MPN ECS80185PX -> ECS-80-18-5PX-TR; Manufacturer_Part_Number (none) -> ECS80185PX
Changed lines of the file:
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@@
 			)
 		)
-		(property "Value" "5V"
+		(property "Value" "TestPoint"
 			(at 266.7 80.0099 90)
 			(effects
@@
 				)
 				(justify left)
+				(hide yes)
 			)
 		)
@@
 			)
 		)
-		(property "MPN" "NANOSMDC075"
+		(property "MPN" "NANOSMDC075F-2"
 			(at 257.048 92.964 0)
 			(effects
@@
 					(color 0 132 132 1)
 				)
+				(hide yes)
 			)
 		)
@@
 			)
 		)
-		(property "Manufacturer_Part_Number" ""
-			(at 248.92 90.17 90)
+		(property "Manufacturer_Part_Number" "NANOSMDC075"
+			(at 257.556 92.71 0)
 			(effects
 				(font
 					(size 1.27 1.27)
+					(color 0 132 132 1)
 				)
-				(hide yes)
 			)
 		)
@@
 			)
 		)
-		(property "MPN" "ECS80185PX"
+		(property "MPN" "ECS-80-18-5PX-TR"
 			(at 58.166 101.6 90)
 			(effects
@@
 					(color 0 132 132 1)
 				)
+				(hide yes)
 			)
 		)
-		(property "Manufacturer_Part_Number" ""
-			(at 50.8 97.79 90)
+		(property "Manufacturer_Part_Number" "ECS80185PX"
+			(at 57.404 101.6 90)
 			(effects
 				(font
 					(size 1.27 1.27)
+					(color 0 132 132 1)
 				)
-				(hide yes)
 			)
 		)
@@
 			)
 		)
-		(property "MPN" "USB3076-30"
+		(property "MPN" "USB3076-30-A"
 			(at 270.764 91.186 0)
 			(effects
@@
 					(color 0 132 132 1)
 				)
+				(hide yes)
 			)
 		)
-		(property "Manufacturer_Part_Number" ""
-			(at 270.51 100.33 0)
+		(property "Manufacturer_Part_Number" "USB3076-30"
+			(at 270.764 91.186 0)
 			(effects
 				(font
 					(size 1.27 1.27)
+					(color 0 132 132 1)
 				)
-				(hide yes)
 			)
 		)

Commit message: SV's comments
Other:
- note added: "Check feasibility for adding pullup 3.3V to D+ USB line"
Changed lines of the file:
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@@
+		)
+	)
+	(text "Check feasibility for adding pullup 3.3V to D+ USB line"
+		(exclude_from_sim no)
+		(at 290.322 82.296 0)
+		(effects
+			(font
+				(size 1.27 1.27)
+				(color 255 7 16 1)
+			)
 		)
 	)

Commit message: All comments addressed
Parts:
- added R71: 0R, Resistor_SMD:R_0603_1608Metric, symbol Device:R_US
- SW5: MPN PTS645SK50SMTR92 LFS -> SWT0310-043016GSA
Connections:
- net +5V: now also R71.2; no longer D8.1 (K)
- new net: D8.1 (K), R71.1
Other:
- note removed: "Check feasibility for adding pullup 3.3V to D+ USB line"
- moved on the sheet: D8, F1, R23, R24, R26, R27, TP5, U4
