File: Main MCU.kicad_sch (KiCad schematic)
At the start: 55 parts, among them J1 F407 SWD, J2 GPIO, J3 Conn_01x02_Pin, SW1 SW_Push, SW2 SW_Push, SW3 SW_Push, SW4 SW_Push, U1 STM32F407VGTx, U2 MCP1825S-3302E/EB

Commit message: Alternate MPNs added
Parts:
- FB1: MPN MPZ1608S601 -> MPZ1608S601ATA00; Manufacturer_Part_Number (none) -> MPZ1608S601
- TP3: value GND -> TestPoint
- TP4: value 3V3 -> TestPoint
Changed lines of the file:
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@@
 			)
 		)
-		(property "Value" "3V3"
+		(property "Value" "TestPoint"
 			(at 274.32 39.3699 90)
 			(effects
@@
 				)
 				(justify left)
+				(hide yes)
 			)
 		)
@@
 			)
 		)
-		(property "MPN" "MPZ1608S601"
+		(property "MPN" "MPZ1608S601ATA00"
 			(at 93.472 29.972 0)
 			(effects
@@
 					(color 0 132 132 1)
 				)
+				(hide yes)
 			)
 		)
@@
 			)
 		)
-		(property "Manufacturer_Part_Number" ""
-			(at 82.55 26.67 0)
-			(effects
-				(font
-					(size 1.27 1.27)
-				)
-				(hide yes)
+		(property "Manufacturer_Part_Number" "MPZ1608S601"
+			(at 93.218 29.972 0)
+			(effects
+				(font
+					(size 1.27 1.27)
+					(color 0 132 132 1)
+				)
 			)
 		)
@@
 			)
 		)
-		(property "Value" "GND"
+		(property "Value" "TestPoint"
 			(at 138.43 190.4999 90)
 			(effects
@@
 				)
 				(justify left)
-			)
-		)
+				(hide yes)
+			)
+		)

Commit message: SV's comments
Other:
- note added: "Add TP"
- note added: "Add actual pins"
- note added: "Check internal pullups if present"
Changed lines of the file:
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@@
+		)
+	)
+	(text "Check internal pullups if present"
+		(exclude_from_sim no)
+		(at 64.516 149.606 0)
+		(effects
+			(font
+				(size 1.27 1.27)
+				(color 255 0 19 1)
+			)
 		)
 	)
@@
 			(font
 				(size 1.27 1.27)
+			)
+		)
+	)
+	(text "Add actual pins"
+		(exclude_from_sim no)
+		(at 48.768 95.25 0)
+		(effects
+			(font
+				(size 1.27 1.27)
+				(color 255 0 7 1)
 			)
 		)
@@
 		)
 	)
+	(text "Add TP"
+		(exclude_from_sim no)
+		(at 94.488 39.878 0)
+		(effects
+			(font
+				(size 1.27 1.27)
+				(color 255 0 65 1)
+			)
+		)
+	)

Commit message: All comments addressed
Parts:
- C18: MPN GRM188R72A102KA01D -> C0603C102K4RACTU
- SW1, SW2, SW3, SW4: MPN PTS645SK50SMTR92 LFS -> SWT0310-043016GSA
Other:
- note added: "(MISO)"
- note added: "(MOSI)"
- note added: "(PWM1)"
- note added: "(PWM2)"
- note added: "(PWM3)"
- note added: "(PWM4)"
- note added: "(RX)"
- note added: "(SCK)"
- note added: "(SCL)"
- note added: "(SDA)"
- note added: "(TX)"
- note removed: "Add TP"
- note removed: "Add actual pins"
- note removed: "Check internal pullups if present"
Changed lines of the file:
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@@
 		)
 	)
-	(text "Check internal pullups if present"
+	(text "(SCL)"
 		(exclude_from_sim no)
-		(at 64.516 149.606 0)
+		(at 27.686 112.268 0)
+		(effects
+			(font
+				(size 1.27 1.27)
+			)
+		)
+	)
+	(text "(PWM3)"
+		(exclude_from_sim no)
+		(at 66.04 119.634 0)
 		(effects
 			(font
 				(size 1.27 1.27)
-				(color 255 0 19 1)
 			)
 		)
@@
 		)
 	)
+	(text "(RX)"
+		(exclude_from_sim no)
+		(at 64.516 124.968 0)
+		(effects
+			(font
+				(size 1.27 1.27)
+			)
+		)
+	)
 	(text "BTN1"
 		(exclude_from_sim no)
@@
 		)
 	)
-	(text "Add actual pins"
+	(text "(MISO)"
 		(exclude_from_sim no)
-		(at 48.768 95.25 0)
+		(at 27.178 122.428 0)
 		(effects
 			(font
 				(size 1.27 1.27)
-				(color 255 0 7 1)
 			)
 		)
@@
 		)
 	)
+	(text "(TX)"
+		(exclude_from_sim no)
+		(at 28.448 124.968 0)
+		(effects
+			(font
+				(size 1.27 1.27)
+			)
+		)
+	)
 	(text "1mA"
 		(exclude_from_sim no)
@@
 		)
 	)
+	(text "(PWM2)"
+		(exclude_from_sim no)
+		(at 65.024 117.094 0)
+		(effects
+			(font
+				(size 1.27 1.27)
+			)
+		)
+	)
 	(text "1.45mA"
 		(exclude_from_sim no)
@@
 		)
 	)
+	(text "(PWM1)"
+		(exclude_from_sim no)
+		(at 65.024 114.554 0)
+		(effects
+			(font
+				(size 1.27 1.27)
+			)
+		)
+	)
+	(text "(PWM4)"
+		(exclude_from_sim no)
+		(at 66.04 122.428 0)
+		(effects
+			(font
+				(size 1.27 1.27)
+			)
+		)
+	)
 	(text "RESET"
 		(exclude_from_sim no)
@@
 		)
 	)
+	(text "(SDA)"
+		(exclude_from_sim no)
+		(at 27.686 114.808 0)
+		(effects
+			(font
+				(size 1.27 1.27)
+			)
+		)
+	)
+	(text "(SCK)"
+		(exclude_from_sim no)
+		(at 27.686 117.348 0)
+		(effects
+			(font
+				(size 1.27 1.27)
+			)
+		)
+	)
 	(text "GPIO Extension"
 		(exclude_from_sim no)
@@
 		)
 	)
-	(text "Peripherals"
+	(text "(MOSI)"
 		(exclude_from_sim no)
-		(at 196.088 113.03 0)
+		(at 27.178 119.888 0)
 		(effects
 			(font
-				(size 2.286 2.286)
+				(size 1.27 1.27)
 			)
-			(justify left bottom)
 		)
 	)
-	(text "Add TP"
+	(text "Peripherals"
 		(exclude_from_sim no)
-		(at 94.488 39.878 0)
+		(at 196.088 113.03 0)
 		(effects
 			(font
-				(size 1.27 1.27)
-				(color 255 0 65 1)
+				(size 2.286 2.286)
 			)
+			(justify left bottom)
 		)
 	)
@@
 			)
 		)
-		(property "Description" "CAP CER 1000PF 100V X7R 0603"
+		(property "Description" "CAP CER 1000PF 16V X7R 0603"
 			(at 203.2 76.2 0)
 			(effects
@@
 			)
 		)
-		(property "MPN" "GRM188R72A102KA01D"
+		(property "MPN" "C0603C102K4RACTU"
 			(at 203.2 76.2 0)
 			(effects
@@
 			)
 		)
-		(property "MPN" "PTS645SK50SMTR92 LFS"
+		(property "MPN" "SWT0310-043016GSA"
 			(at 41.91 55.88 90)
 			(effects
@@
 			)
 		)
-		(property "MPN" "PTS645SK50SMTR92 LFS"
+		(property "MPN" "SWT0310-043016GSA"
 			(at 25.4 44.45 90)
 			(effects
@@
 			)
 		)
-		(property "MPN" "PTS645SK50SMTR92 LFS"
+		(property "MPN" "SWT0310-043016GSA"
 			(at 227.33 127 90)
 			(effects
@@
 			)
 		)
-		(property "MPN" "PTS645SK50SMTR92 LFS"
+		(property "MPN" "SWT0310-043016GSA"
 			(at 207.01 127 90)
 			(effects
